Commit message: rename outdoor kurt_base refs, too

File: urdf/kurt_outdoor.urdf.xacro (robot description, xacro)
@@ -6,5 +6,5 @@
   name="kurt_outdoor_base">
   <xacro:include filename="$(find uos_common_urdf)/common.xacro" />
-  <xacro:include filename="$(find kurt_base)/urdf/infrared_sonar.urdf.xacro" />
+  <xacro:include filename="$(find kurtberry_pi)/urdf/infrared_sonar.urdf.xacro" />
   <xacro:include filename="$(find uos_common_urdf)/urdf/imu.gazebo.urdf.xacro" />
   <xacro:property name="wheel_width" value="0.046" />
@@ -21,5 +21,5 @@
       <origin xyz="0 0 0" rpy="0 0 0" />
       <geometry>
-        <mesh filename="package://kurt_base/meshes/kurt_base_outdoor.stl" />
+        <mesh filename="package://kurtberry_pi/meshes/kurt_base_outdoor.stl" />
       </geometry>
       <material name="red" >
@@ -30,5 +30,5 @@
       <origin xyz="0 0 0" rpy="0 0 0" />
       <geometry>
-        <mesh filename="package://kurt_base/meshes/kurt_base_outdoor.stl" />
+        <mesh filename="package://kurtberry_pi/meshes/kurt_base_outdoor.stl" />
       </geometry>
     </collision>
@@ -91,5 +91,5 @@
         <origin xyz="0 0 0" rpy="0 0 0" />
         <geometry>
-          <mesh filename="package://kurt_base/meshes/kurt_wheel_outdoor.stl" />
+          <mesh filename="package://kurtberry_pi/meshes/kurt_wheel_outdoor.stl" />
         </geometry>
         <material name="blackish"><color rgba="0.1 0.1 0.1 1"/></material>
@@ -98,5 +98,5 @@
         <origin xyz="0 0 0" rpy="0 0 0" />
         <geometry>
-          <mesh filename="package://kurt_base/meshes/kurt_wheel_outdoor.stl" />
+          <mesh filename="package://kurtberry_pi/meshes/kurt_wheel_outdoor.stl" />
           <!-- <cylinder length="${wheel_width}" radius="${wheel_radius}" /> -->
         </geometry>
